File: inboard386/inboard386.kicad_sch (KiCad schematic)
At the start: 199 parts, among them J1 Conn_02x20_Odd_Even, J2 Conn_02x20_Odd_Even, J3 CPU_Cable, J4 Bus_ISA_8bit, U1 TMM41256AP, U10 TMM41256AP, U100 PAL16L8, U101 TIBPAL16R4, U102 TIBPAL16R6, U11 TMM41256AP, U12 TMM41256AP, U13 TMM41256AP, U14 TMM41256AP, U15 TMM41256AP, U16 TMM41256AP, U17 TMM41256AP, U18 TMM41256AP, U19 TMM41256AP, U2 TMM41256AP, U20 TMM41256AP, U21 TMM41256AP, U22 TMM41256AP, U23 TMM41256AP, U24 TMM41256AP, U25 TMM41256AP, U26 TMM41256AP, U27 TMM41256AP, U28 TMM41256AP, U29 TMM41256AP, U3 TMM41256AP, U30 TMM41256AP, U31 TMM41256AP, U32 TMM41256AP, U33 TMM41256AP, U34 TMM41256AP, U35 TMM41256AP, U36 TMM41256AP, U37 74F280, U38 74F280, U39 74AS1004, U4 TMM41256AP, U40 74F280, U41 74AS1004, U42 74AS1032, U43 74AS1032, U44 74F280, U45 74F74, U46 74ALS244, U47 74ALS373, U48 74ALS244, U49 74ALS373, U5 TMM41256AP, U50 74ALS244, U51 74ALS373, U52 74ALS373, U53 74ALS244, U54 74F244, U55 74ALS245, U56 74ALS245, U57 74ALS245, U58 74F32, U59 74AS21, U6 TMM41256AP, U60 74F00, U61 74F258, U62 74F74, U63 74F74, U64 74F258, U65 74AS1000, U66 74F74, U67 74F74, U68 74F153, U69 74LS174, U7 TMM41256AP, U70 PAL16R8, U71 PAL20L8, U72 74ALS245, U73 80386, U74 PAL16R4, U75 PAL16R6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

Commit message: update signal names in schematic and logic, add prototype logic for 8MB ram expansion
Connections:
- net ROMCACHE: now reaches U101.7 (I_{6}), U69.2 (Q0), U71.14 (I_{11})
- net ~{RAS_EN_SYS}: now reaches U42.5, U43.5, U71.20 (I/~{O_{6}})
- net ~{RAS_EN_4M}: now reaches J2.15 (Pin_15), U71.15 (~{O_{1}})
- net ~{RAS_EN_1M_2}: now reaches J2.18 (Pin_18), U71.22 (~{O_{8}})
- net ~{RAS_EN_1M_1}: now reaches J2.19 (Pin_19), U71.21 (I/~{O_{7}})
Changed lines of the file:
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@@
 	)
 	(junction
-		(at 273.05 803.91)
-		(diameter 0)
-		(color 0 0 0 0)
-	)
-	(junction
 		(at 769.62 389.89)
 		(diameter 0)
@@
 	(wire
 		(pts
-			(xy 93.98 805.18) (xy 99.06 805.18)
-		)
-		(stroke
-			(width 0)
-			(type default)
-		)
-	)
-	(wire
-		(pts
 			(xy 656.59 683.26) (xy 656.59 775.97)
 		)
@@
 	(wire
 		(pts
-			(xy 273.05 803.91) (xy 273.05 655.32)
-		)
-		(stroke
-			(width 0)
-			(type default)
-		)
-	)
-	(wire
-		(pts
 			(xy 816.61 358.14) (xy 820.42 358.14)
 		)
@@
 	(wire
 		(pts
-			(xy 273.05 803.91) (xy 533.4 803.91)
-		)
-		(stroke
-			(width 0)
-			(type default)
-		)
-	)
-	(wire
-		(pts
 			(xy 383.54 101.6) (xy 383.54 114.3)
 		)
@@
 	(wire
 		(pts
-			(xy 273.05 655.32) (xy 266.7 655.32)
-		)
-		(stroke
-			(width 0)
-			(type default)
-		)
-	)
-	(wire
-		(pts
 			(xy 325.12 694.69) (xy 325.12 718.82)
 		)
@@
 	(wire
 		(pts
-			(xy 273.05 803.91) (xy 273.05 825.5)
-		)
-		(stroke
-			(width 0)
-			(type default)
-		)
-	)
-	(wire
-		(pts
 			(xy 422.91 350.52) (xy 422.91 322.58)
 		)
@@
 	(wire
 		(pts
-			(xy 273.05 825.5) (xy 93.98 825.5)
-		)
-		(stroke
-			(width 0)
-			(type default)
-		)
-	)
-	(wire
-		(pts
 			(xy 427.99 360.68) (xy 427.99 312.42)
 		)
@@
 	(wire
 		(pts
-			(xy 93.98 825.5) (xy 93.98 805.18)
-		)
-		(stroke
-			(width 0)
-			(type default)
-		)
-	)
-	(wire
-		(pts
 			(xy 659.13 363.22) (xy 668.02 363.22)
 		)
@@
 		)
 	)
+	(label "~{RAS_EN_1M_2}"
+		(at 554.99 793.75 0)
+		(effects
+			(font
+				(size 1.27 1.27)
+			)
+			(justify left bottom)
+		)
+	)
+	(label "~{RAS_EN_4M}"
+		(at 554.99 775.97 0)
+		(effects
+			(font
+				(size 1.27 1.27)
+			)
+			(justify left bottom)
+		)
+	)
 	(label "~{MUX_BE3}"
 		(at 389.89 406.4 0)
@@
 		)
 	)
+	(label "~{RAS_EN_1M_1}"
+		(at 554.99 791.21 0)
+		(effects
+			(font
+				(size 1.27 1.27)
+			)
+			(justify left bottom)
+		)
+	)
 	(label "~{MUX_BE0}"
 		(at 382.27 388.62 0)
@@
 		)
 	)
+	(label "~{RAS_EN_SYS}"
+		(at 554.99 788.67 0)
+		(effects
+			(font
+				(size 1.27 1.27)
+			)
+			(justify left bottom)
+		)
+	)
 	(label "~{MUX_BE1}"
 		(at 389.89 401.32 0)
@@
 		)
 	)
+	(global_label "ROMCACHE"
+		(shape input)
+		(at 266.7 655.32 90)
+		(fields_autoplaced yes)
+		(effects
+			(font
+				(size 1.27 1.27)
+			)
+			(justify left)
+		)
+		(property "Intersheetrefs" "${INTERSHEET_REFS}"
+			(at 266.7 642.1748 90)
+			(hide yes)
+			(show_name no)
+			(do_not_autoplace no)
+			(effects
+				(font
+					(size 1.27 1.27)
+				)
+				(justify left)
+			)
+		)
+	)
 	(global_label "~{CAS0}"
 		(shape input)
@@
 		)
 	)
+	(global_label "ROMCACHE"
+		(shape input)
+		(at 533.4 803.91 180)
+		(fields_autoplaced yes)
+		(effects
+			(font
+				(size 1.27 1.27)
+			)
+			(justify right)
+		)
+		(property "Intersheetrefs" "${INTERSHEET_REFS}"
+			(at 520.2548 803.91 0)
+			(hide yes)
+			(show_name no)
+			(do_not_autoplace no)
+			(effects
+				(font
+					(size 1.27 1.27)
+				)
+				(justify right)
+			)
+		)
+	)
 	(global_label "8088_AD0"
 		(shape input)
@@
 			)
 		)
+	)
+	(global_label "ROMCACHE"
+		(shape input)
+		(at 99.06 805.18 180)
+		(fields_autoplaced yes)
+		(effects
+			(font
+				(size 1.27 1.27)
+			)
+			(justify right)
+		)
+		(property "Intersheetrefs" "${INTERSHEET_REFS}"
+			(at 85.9148 805.18 0)
+			(hide yes)
+			(show_name no)
+			(do_not_autoplace no)
+			(effects
+				(font
+					(size 1.27 1.27)
+				)
+				(justify right)
+			)
+		)
