File: inboard386/inboard386.kicad_pcb (KiCad board)
At the start: 6 copper layers, 338.8 x 107.2 mm, 199 parts, among them J1 Conn_02x20_Odd_Even, J2 Conn_02x20_Odd_Even, J3 CPU_Cable, J4 Bus_ISA_8bit, U1 TMM41256AP, U10 TMM41256AP, U100 PAL16L8, U101 TIBPAL16R4, U102 TIBPAL16R6, U11 TMM41256AP, U12 TMM41256AP, U13 TMM41256AP, U14 TMM41256AP, U15 TMM41256AP, U16 TMM41256AP, U17 TMM41256AP, U18 TMM41256AP, U19 TMM41256AP, U2 TMM41256AP, U20 TMM41256AP, U21 TMM41256AP, U22 TMM41256AP, U23 TMM41256AP, U24 TMM41256AP, U25 TMM41256AP, U26 TMM41256AP, U27 TMM41256AP, U28 TMM41256AP, U29 TMM41256AP, U3 TMM41256AP, U30 TMM41256AP, U31 TMM41256AP, U32 TMM41256AP, U33 TMM41256AP, U34 TMM41256AP, U35 TMM41256AP, U36 TMM41256AP, U37 74F280, U38 74F280, U39 74AS1004, U4 TMM41256AP, U40 74F280, U41 74AS1004, U42 74AS1032, U43 74AS1032, U44 74F280, U45 74F74, U46 74ALS244, U47 74ALS373, U48 74ALS244, U49 74ALS373, U5 TMM41256AP, U50 74ALS244, U51 74ALS373, U52 74ALS373, U53 74ALS244, U54 74F244, U55 74ALS245, U56 74ALS245, U57 74ALS245, U58 74F32, U59 74AS21, U6 TMM41256AP, U60 74F00, U61 74F258, U62 74F74, U63 74F74, U64 74F258, U65 74AS1000, U66 74F74, U67 74F74, U68 74F153, U69 74LS174, U7 TMM41256AP, U70 PAL16R8, U71 PAL20L8, U72 74ALS245, U73 80386, U74 PAL16R4, U75 PAL16R6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

Commit message: update signal names in schematic and logic, add prototype logic for 8MB ram expansion
Parts:
- moved J1 0.13 mm to (38.6, 67.9)
- moved J2 0.13 mm to (152.9, 67.9)
Other:
- board text added: "rev. 0.1a"
- board text removed: "rev. 0.1"
